File: tja1050_breakout.kicad_pcb (KiCad board)
At the start: 2 copper layers, 32.2 x 15.7 mm, 11 parts, among them J1 Termination Jumper, J2 CAN Jumper, J3 Phoenix Block, J4 Jumper, J5 CANS Jumper, U1 TJA1051T

Commit message: add vias
Routing:
- net GND: track 18.3 -> 6.64 mm, vias 0 -> 2
Changed lines of the file:
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@@
 	)
 	(segment
-		(start 99.81 92.044999)
-		(end 98.355 92.044999)
+		(start 105.2 90.12)
+		(end 105.2 90.88)
 		(width 0.5)
 		(layer "F.Cu")
@@
 	)
 	(segment
-		(start 105.2 90.12)
-		(end 104.7 89.62)
-		(width 0.5)
-		(layer "F.Cu")
-		(net 1)
-	)
-	(segment
-		(start 104.7 89.62)
-		(end 102.234999 89.62)
-		(width 0.5)
-		(layer "F.Cu")
-		(net 1)
-	)
-	(segment
-		(start 105.18 95.994998)
+		(start 105.18 95)
 		(end 105.18 94.41)
 		(width 0.5)
@@
 	)
 	(segment
-		(start 103.339999 97.834999)
-		(end 105.18 95.994998)
-		(width 0.5)
-		(layer "F.Cu")
-		(net 1)
-	)
-	(segment
 		(start 98.355 92.044999)
 		(end 96.55 92.044999)
-		(width 0.5)
-		(layer "F.Cu")
-		(net 1)
-	)
-	(segment
-		(start 102.234999 89.62)
-		(end 99.81 92.044999)
-		(width 0.5)
-		(layer "F.Cu")
-		(net 1)
-	)
-	(segment
-		(start 105.2 90.88)
-		(end 105.2 90.12)
 		(width 0.5)
 		(layer "F.Cu")
@@
 		(net 1)
 	)
+	(via
+		(at 105.18 95)
+		(size 0.6)
+		(drill 0.3)
+		(layers "F.Cu" "B.Cu")
+		(net 1)
+	)
+	(via
+		(at 105.2 90.12)
+		(size 0.6)
+		(drill 0.3)
+		(layers "F.Cu" "B.Cu")
+		(net 1)
+	)

Commit message: update schematic
Parts:
- J2: value CAN Jumper -> Phoenix Block
- J3: value Phoenix Block -> CAN Jumper
Changed lines of the file:
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@@
 			)
 		)
-		(property "Value" "CAN Jumper"
+		(property "Value" "Phoenix Block"
 			(at 2.54 5.72 90)
 			(layer "F.Fab")
@@
 			)
 		)
-		(property "Value" "Phoenix Block"
+		(property "Value" "CAN Jumper"
 			(at 0 4.92 0)
 			(layer "F.Fab")

Commit message: v1.1 initial
Parts:
- C1, C2, C3: footprint Capacitor_SMD:C_0402_1005Metric -> Capacitor_SMD:C_0603_1608Metric
- R1: footprint Resistor_SMD:R_0402_1005Metric -> Resistor_SMD:R_0603_1608Metric
- moved J1 1.07 mm to (106.9, 87.8)
- moved R1 0.95 mm to (106.9, 91.2)
- moved C1 0.54 mm to (105.4, 94.2)
- moved C2 0.43 mm to (105.4, 91.2)
- moved C3 0.25 mm to (96.2, 92.7)
Routing:
- net /CAN+: track 17.1 -> 15.6 mm
- net /CAN-: track 33.6 -> 32.4 mm
Other:
- board text added: "CAN_H"
- board text added: "CAN_L"
- board text removed: "CANH"
- board text removed: "CANL"
